File: pcb/window-contact-rfm69.kicad_pcb (KiCad board)
At the start: 2 copper layers, 38.4 x 41.2 mm, 10 parts, among them IC1 ATMEGA328P-P, P1 REED, P2 BME280, P3 AN

Commit message: changed to tqfp atmel
Parts:
- removed BT1: CR2477, battery:CR2477
- removed C1: 100nf, Capacitors_SMD:C_0805_HandSoldering
- removed C2: 10uF, Capacitors_SMD:c_elec_4x5.8
- removed IC1: ATMEGA328P-P, Housings_DIP:DIP-28_W7.62mm
- removed P1: REED, Pin_Headers:Pin_Header_Straight_1x03
- removed P2: BME280, Pin_Headers:Pin_Header_Straight_1x04
- removed P3: AN, Wire_Pads:SolderWirePad_single_1mmDrill
- removed R1: 10k, Resistors_SMD:R_0805_HandSoldering
- removed R2: 10M, Resistors_ThroughHole:Resistor_Horizontal_RM10mm
- removed RF1: RFM69, rfm69:RFM96
Routing:
- net VCC: track 114.4 -> 0.00 mm, vias 5 -> 0
- net GND: track 101.0 -> 0.00 mm, vias 4 -> 0
- net Net-(IC1-Pad4): track 39.0 -> 0.00 mm, vias 4 -> 0
- net Net-(IC1-Pad5): track 31.5 -> 0.00 mm
- net Net-(IC1-Pad28): track 28.6 -> 0.00 mm
- net Net-(IC1-Pad27): track 28.5 -> 0.00 mm, vias 1 -> 0
- net Net-(IC1-Pad18): track 27.7 -> 0.00 mm, vias 2 -> 0
- net Net-(IC1-Pad16): track 23.7 -> 0.00 mm, vias 2 -> 0
- net Net-(IC1-Pad17): track 11.6 -> 0.00 mm
- net Net-(IC1-Pad19): track 9.73 -> 0.00 mm
- net Net-(P3-Pad1): track 6.26 -> 0.00 mm
- net Net-(IC1-Pad1): track 3.56 -> 0.00 mm
Other:
- board outline removed

Commit message: updated kicad files
Parts:
- added BT1: CR2477, battery:CR2477, F.Cu at (152.2, 134.6)
- added C1: 10uF, Capacitors_SMD:c_elec_4x5.8, F.Cu at (164.2, 123.2)
- added C2: 100nf, Capacitors_SMD:C_0805_HandSoldering, B.Cu at (157.0, 122.8)
- added C3: 100nf, Capacitors_SMD:C_0805_HandSoldering, F.Cu at (148.6, 118.6)
- added IC1: ATMEGA328P-A, Housings_QFP:TQFP-32_7x7mm_Pitch0.8mm, B.Cu at (148.8, 120.0)
- added P1: VCC, wirepad:Wire_SMD_Pad_1PIN, F.Cu at (141.2, 114.2)
- added P2: TX/RX, Pin_Headers:Pin_Header_Straight_1x02, F.Cu at (140.6, 122.0)
- added P3: RE1, wirepad:Wire_SMD_Pad_1PIN, F.Cu at (155.6, 114.2)
- added P4: ISP, isp:SMD, B.Cu at (155.8, 143.6)
- added P5: RE2, wirepad:Wire_SMD_Pad_1PIN, F.Cu at (157.8, 114.2)
- added P6: AN, Wire_Pads:SolderWirePad_single_1mmDrill, F.Cu at (140.2, 125.6)
- added R1: 10k, Resistors_SMD:R_0805_HandSoldering, B.Cu at (140.2, 130.6)
- added R2: 10M, Resistors_SMD:R_0805_HandSoldering, F.Cu at (163.8, 117.2)
- added R3: 10M, Resistors_SMD:R_0805_HandSoldering, F.Cu at (161.2, 117.2)
- added R4: 1k, Resistors_SMD:R_0805_HandSoldering, B.Cu at (156.8, 146.4)
- added R5: 1k, Resistors_SMD:R_0805_HandSoldering, B.Cu at (162.2, 129.8)
- added R6: 1k, Resistors_SMD:R_0805_HandSoldering, B.Cu at (143.4, 139.2)
- added RF1: RFM69, rfm69:RFM96, B.Cu at (153.8, 143.0)
Routing:
- net GND: track 0.00 -> 114.9 mm, vias 0 -> 10
- net VCC: track 0.00 -> 97.6 mm, vias 0 -> 5
- net /MOSI: track 0.00 -> 43.9 mm, vias 0 -> 6
- net /SCK: track 0.00 -> 43.1 mm, vias 0 -> 4
- net Net-(IC1-Pad32): track 0.00 -> 37.5 mm, vias 0 -> 4
- net Net-(IC1-Pad24): track 0.00 -> 32.7 mm, vias 0 -> 3
- net Net-(IC1-Pad29): track 0.00 -> 31.3 mm, vias 0 -> 2
- net /MISO: track 0.00 -> 29.7 mm, vias 0 -> 4
- net Net-(R6-Pad2): track 0.00 -> 22.6 mm, vias 0 -> 2
- net Net-(IC1-Pad23): track 0.00 -> 19.0 mm, vias 0 -> 3
- net /SS: track 0.00 -> 14.2 mm, vias 0 -> 2
- net Net-(P6-Pad1): track 0.00 -> 8.61 mm
- net Net-(R5-Pad2): track 0.00 -> 8.36 mm
- net Net-(IC1-Pad30): track 0.00 -> 6.21 mm, vias 0 -> 1
- net Net-(IC1-Pad31): track 0.00 -> 4.61 mm, vias 0 -> 1
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- added copper zone on F.Cu, net GND
Other:
- board outline added: 28.2 x 34 mm
